Commit message: Pristine configuration files as provided by user.

File: cartographer_ros/urdf/backpack_3d.urdf (robot description, URDF)
Before this commit: robot cartographer_backpack_3d, 4 links, 3 joints
Links:
- removed link horizontal_vlp16_link
- removed link imu_link
- added link imu; visual box size=0.06 0.04 0.02
- added link velodyne; visual cylinder length=0.07 radius=0.05
Joints:
- removed joint horizontal_vlp16_link_joint
- added joint velodyne_link_joint: type fixed, parent base_link, child velodyne, origin xyz=-0.0088 -0.0205 0.12562 rpy=0. 0. 0.
- joint imu_link_joint: child imu_link -> imu

Commit message: Pristine config files as desribed by the user

File: cartographer_ros/urdf/backpack_3d.urdf (robot description, URDF)
Before this commit: robot cartographer_backpack_3d, 4 links, 3 joints
Links:
- removed link horizontal_vlp16_link
- removed link vertical_vlp16_link
- added link rslidar; visual cylinder length=0.07 radius=0.05
Joints:
- removed joint vertical_vlp16_link_joint
- joint horizontal_vlp16_link_joint: child horizontal_vlp16_link -> rslidar
